File: Documentation/Kicad/F1/PS2-MSX-F1.sch (KiCad schematic (older format))
At the start: 31 parts, among them J1 Conn_02x17_Odd_Even, J2 Conn_01x04, J3 Conn_01x04, Q1 2SC1815, Q2 2N2907, U1 STM32F103C6T6 BluePill

Commit message: NPN base resistor update
Parts:
- R10: value 33K -> 5K6
Changed lines of the file:
@@
 P 8300 3150
 F 0 "R10" V 8300 3050 50  0000 L CNN
-F 1 "33K" V 8200 3050 50  0000 L CNN
+F 1 "5K6" V 8200 3050 50  0000 L CNN
 F 2 "Resistor_THT:R_Axial_DIN0204_L3.6mm_D1.6mm_P7.62mm_Horizontal" V 8230 3150 50  0001 C CNN
 F 3 "~" H 8300 3150 50  0001 C CNN
