File: Documentation/Kicad/F1/PS2-MSX-F1.kicad_pcb (KiCad board)
At the start: 2 copper layers, 55 x 65 mm, 35 parts, among them J1 Conn_02x17_Odd_Even, J2 Conn_01x04, J3 Conn_01x04, Q1 2SC1815, Q2 2N2907, U1 STM32F103C6T6 BluePill

Commit message: Documentation update
Documentation update
Other:
- board text added: "PS/2 to MSX keyboard interface F1 v1.0"
- board text removed: "PS/2 to MSX keyboard interface vF1"
