File: Documentation/Kicad/F4/PS2-MSX-F4.sch (KiCad schematic (older format))
At the start: 30 parts, among them J1 Conn_02x17_Odd_Even, J2 Conn_01x04, J3 Conn_01x04, Q1 2SC1815, Q2 2N2907, U1 WeAct Studio STM32F401CEU6 V3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

Commit message: Documentation update
Parts:
- R10: value 33K -> 5K6
Connections:
- net PS2Clk: now also U1.15 (PB7)
- net X0': now also R1.2, U1.1 (PB12)
- no-connect marks 18 -> 17
